File: Schaltplan_embedded/KiCad/ES_proj_LoRaWAN_fsm/Schaltplan_embedded.sch (KiCad schematic (older format))
At the start: 0 parts

Commit message: schaltplan neu
Changed lines of the file:
@@
 $EndSheet
 $Sheet
-S 4450 1050 3550 1250
+S 4450 1100 3550 1250
 U 5E150549
-F0 "Peripherie" 50
-F1 "Peripherie.sch" 50
+F0 "Sensorik" 50
+F1 "Sensorik.sch" 50
 $EndSheet
 $EndSCHEMATC

Commit message: Neuer Schaltplan
Changed lines of the file:
@@
 $EndDescr
 $Sheet
-S 950  850  3100 1550
+S 950  800  3100 1550
 U 5DC1A511
 F0 "Microcontroller" 50
