File: Schaltplan_embedded/KiCad/ES_proj_LoRaWAN_fsm/Microcontroller.sch (KiCad schematic (older format))
At the start: 16 parts, among them J1 Conn_02x05_Odd_Even, J7 Conn_01x02, U1 STM32L476RGTx, Y1 Crystal 8Mhz

Commit message: so
Parts:
- renumbered C2 to C1, C1 to C2, J7 to J2
Connections:
- no-connect marks 17 -> 18
Changed lines of the file:
@@
 $EndDescr
 $Comp
-L power:GND #PWR0101
+L power:GND #PWR01
 U 1 1 5DC1A6C7
 P 1600 4650
-F 0 "#PWR0101" H 1600 4400 50  0001 C CNN
+F 0 "#PWR01" H 1600 4400 50  0001 C CNN
 F 1 "GND" H 1605 4477 50  0000 C CNN
 F 2 "" H 1600 4650 50  0001 C CNN
@@
 $EndComp
 $Comp
-L Device:C C1
+L Device:C C2
 U 1 1 5DC1A815
 P 1950 4500
-F 0 "C1" H 2065 4546 50  0000 L CNN
+F 0 "C2" H 2065 4546 50  0000 L CNN
 F 1 "20pF" H 2065 4455 50  0000 L CNN
 F 2 "Capacitors_SMD:C_0603_HandSoldering" H 1988 4350 50  0001 C CNN
@@
 $EndComp
 $Comp
-L power:GND #PWR0102
+L power:GND #PWR04
 U 1 1 5DC1AD63
 P 4100 6650
-F 0 "#PWR0102" H 4100 6400 50  0001 C CNN
+F 0 "#PWR04" H 4100 6400 50  0001 C CNN
 F 1 "GND" H 4105 6477 50  0000 C CNN
 F 2 "" H 4100 6650 50  0001 C CNN
@@
 Connection ~ 6100 1300
 $Comp
-L power:GND #PWR0103
+L power:GND #PWR06
 U 1 1 5DC1EF80
 P 5200 1850
-F 0 "#PWR0103" H 5200 1600 50  0001 C CNN
+F 0 "#PWR06" H 5200 1600 50  0001 C CNN
 F 1 "GND" H 5205 1677 50  0000 C CNN
 F 2 "" H 5200 1850 50  0001 C CNN
@@
 JTAG_RESET
 $Comp
-L power:GND #PWR0104
+L power:GND #PWR09
 U 1 1 5DC3289B
 P 7250 4650
-F 0 "#PWR0104" H 7250 4400 50  0001 C CNN
+F 0 "#PWR09" H 7250 4400 50  0001 C CNN
 F 1 "GND" H 7255 4477 50  0000 C CNN
 F 2 "" H 7250 4650 50  0001 C CNN
@@
 JTAG_RESET
 $Comp
-L power:GND #PWR0105
+L power:GND #PWR011
 U 1 1 5DC3DBCE
 P 8400 3150
-F 0 "#PWR0105" H 8400 2900 50  0001 C CNN
+F 0 "#PWR011" H 8400 2900 50  0001 C CNN
 F 1 "GND" H 8405 2977 50  0000 C CNN
 F 2 "" H 8400 3150 50  0001 C CNN
@@
 $EndComp
 $Comp
-L power:GND #PWR0107
+L power:GND #PWR02
 U 1 1 5DC52E14
 P 2700 3350
-F 0 "#PWR0107" H 2700 3100 50  0001 C CNN
+F 0 "#PWR02" H 2700 3100 50  0001 C CNN
 F 1 "GND" H 2705 3177 50  0000 C CNN
 F 2 "" H 2700 3350 50  0001 C CNN
@@
 $EndComp
 $Comp
-L power:GND #PWR0108
+L power:GND #PWR012
 U 1 1 5DC8150A
 P 9850 4350
-F 0 "#PWR0108" H 9850 4100 50  0001 C CNN
+F 0 "#PWR012" H 9850 4100 50  0001 C CNN
 F 1 "GND" H 9855 4177 50  0000 C CNN
 F 2 "" H 9850 4350 50  0001 C CNN
@@
 	4800 5550 5100 5550
 $Comp
-L power:+3.3V #PWR0114
+L power:+3.3V #PWR03
 U 1 1 5DEBFF94
 P 3900 2600
-F 0 "#PWR0114" H 3900 2450 50  0001 C CNN
+F 0 "#PWR03" H 3900 2450 50  0001 C CNN
 F 1 "+3.3V" H 3915 2773 50  0000 C CNN
 F 2 "" H 3900 2600 50  0001 C CNN
@@
 $EndComp
 $Comp
-L power:+3.3V #PWR0115
+L power:+3.3V #PWR010
 U 1 1 5DEC0739
 P 8400 2050
-F 0 "#PWR0115" H 8400 1900 50  0001 C CNN
+F 0 "#PWR010" H 8400 1900 50  0001 C CNN
 F 1 "+3.3V" H 8415 2223 50  0000 C CNN
 F 2 "" H 8400 2050 50  0001 C CNN
@@
 $EndComp
 $Comp
-L power:+3.3V #PWR0116
+L power:+3.3V #PWR05
 U 1 1 5DEC0C78
 P 5200 1150
-F 0 "#PWR0116" H 5200 1000 50  0001 C CNN
+F 0 "#PWR05" H 5200 1000 50  0001 C CNN
 F 1 "+3.3V" H 5215 1323 50  0000 C CNN
 F 2 "" H 5200 1150 50  0001 C CNN
@@
 $EndComp
 $Comp
-L power:+3.3V #PWR0117
+L power:+3.3V #PWR07
 U 1 1 5DEC1290
 P 5950 4050
-F 0 "#PWR0117" H 5950 3900 50  0001 C CNN
+F 0 "#PWR07" H 5950 3900 50  0001 C CNN
 F 1 "+3.3V" H 5965 4223 50  0000 C CNN
 F 2 "" H 5950 4050 50  0001 C CNN
@@
 	6100 1750 6550 1750
 $Comp
-L power:GND #PWR0106
+L power:GND #PWR08
 U 1 1 5DC3DC91
 P 7200 3050
-F 0 "#PWR0106" H 7200 2800 50  0001 C CNN
+F 0 "#PWR08" H 7200 2800 50  0001 C CNN
 F 1 "GND" H 7205 2877 50  0000 C CNN
 F 2 "" H 7200 3050 50  0001 C CNN
@@
 	3000 5150 3400 5150
 $Comp
-L Connector_Generic:Conn_01x02 J7
+L Connector_Generic:Conn_01x02 J2
 U 1 1 5DE2967D
 P 6950 5200
-F 0 "J7" H 7030 5192 50  0000 L CNN
+F 0 "J2" H 7030 5192 50  0000 L CNN
 F 1 "Conn_01x02" H 7030 5101 50  0000 L CNN
 F 2 "Pin_Headers:Pin_Header_Straight_1x02_Pitch1.00mm" H 6950 5200 50  0001 C CNN
@@
 	6550 5300 6750 5300
 $Comp
-L Device:C C2
+L Device:C C1
 U 1 1 5DC1A899
 P 1950 4050
-F 0 "C2" H 2065 4096 50  0000 L CNN
+F 0 "C1" H 2065 4096 50  0000 L CNN
 F 1 "20pF" H 2065 4005 50  0000 L CNN
 F 2 "Capacitors_SMD:C_0603_HandSoldering" H 1988 3900 50  0001 C CNN
@@
 Wire Wire Line
 	2100 4500 2450 4500
+NoConn ~ 4550 4950
 $EndSCHEMATC

Commit message: Schaltplan nuevo
Parts:
- J2: footprint Pin_Headers:Pin_Header_Straight_1x02_Pitch1.00mm -> Pin_Headers:Pin_Header_Straight_1x02_Pitch2.54mm
Changed lines of the file:
@@
 F 0 "J2" H 7030 5192 50  0000 L CNN
 F 1 "Conn_01x02" H 7030 5101 50  0000 L CNN
-F 2 "Pin_Headers:Pin_Header_Straight_1x02_Pitch1.00mm" H 6950 5200 50  0001 C CNN
+F 2 "Pin_Headers:Pin_Header_Straight_1x02_Pitch2.54mm" H 6950 5200 50  0001 C CNN
 F 3 "~" H 6950 5200 50  0001 C CNN
 	1    6950 5200

Commit message: neuer Schaltplan
Parts:
- S1: symbol Schaltplan_embedded-rescue:LL3301NF065QG-SamacSys_Parts -> Schaltplan_embedded-rescue:LL3301NF065QG-SamacSys_Parts-Schaltplan_embedded-rescue
Connections:
- net GND: now also C4.2
Changed lines of the file:
@@
 $EndComp
 Wire Wire Line
-	5200 1750 6100 1750
+	5200 1750 5650 1750
 Wire Wire Line
 	8100 2800 8200 2800
 $Comp
-L Schaltplan_embedded-rescue:LL3301NF065QG-SamacSys_Parts S1
+L Schaltplan_embedded-rescue:LL3301NF065QG-SamacSys_Parts-Schaltplan_embedded-rescue S1
 U 1 1 5DE990BE
 P 7300 2800
@@
 	2100 4500 2450 4500
 NoConn ~ 4550 4950
+Wire Wire Line
+	5650 1700 5650 1750
+Connection ~ 5650 1750
+Wire Wire Line
+	5650 1750 6100 1750
 $EndSCHEMATC

Commit message: Ruteado semi listo
Connections:
- net AntOFF: now also U1.16 (PA2); no longer U1.61 (PB8)
- no-connect marks 18 -> 22
Changed lines of the file:
@@
 NoConn ~ 3400 4750
 NoConn ~ 4800 4950
-NoConn ~ 4800 3250
 Text GLabel 3100 3050 0    50   Input ~ 0
 JTAG_RESET
@@
 	4400 2750 4400 2850
 Connection ~ 4300 2750
-Text GLabel 5100 5550 2    50   Output ~ 0
+Text GLabel 5100 3250 2    50   Output ~ 0
 AntOFF
-Wire Wire Line
-	4800 5550 5100 5550
 $Comp
 L power:+3.3V #PWR03
@@
 Wire Wire Line
 	2100 4500 2450 4500
-NoConn ~ 4550 4950
 Wire Wire Line
 	5650 1700 5650 1750
@@
 Wire Wire Line
 	5650 1750 6100 1750
+NoConn ~ 4800 3450
+NoConn ~ 4800 5650
+NoConn ~ 4800 5750
+NoConn ~ 4800 5850
+NoConn ~ 4800 5950
+Wire Wire Line
+	4800 3250 5100 3250
+NoConn ~ 4800 5550
 $EndSCHEMATC

Commit message: Neue platine
Connections:
- net LED_OUT: now also U1.9 (PC1); no longer U1.40 (PC9)
- net AntOFF: no longer names the net of U1.16 (PA2)
- no-connect marks 22 -> 23
Changed lines of the file:
@@
 Wire Wire Line
 	2700 3250 2700 3350
-Text GLabel 3000 5650 0    50   Output ~ 0
+Text GLabel 3000 4850 0    50   Output ~ 0
 LED_OUT
 Text GLabel 8600 4350 0    50   Input ~ 0
@@
 NoConn ~ 3400 5050
 NoConn ~ 3400 4950
-NoConn ~ 3400 4850
 NoConn ~ 3400 4750
 NoConn ~ 4800 4950
@@
 	4400 2750 4400 2850
 Connection ~ 4300 2750
-Text GLabel 5100 3250 2    50   Output ~ 0
-AntOFF
 $Comp
 L power:+3.3V #PWR03
@@
 Wire Wire Line
 	4800 3850 5100 3850
-Wire Wire Line
-	3000 5650 3400 5650
 $Comp
 L MCU_ST_STM32L4:STM32L476RGTx U1
@@
 NoConn ~ 4800 5850
 NoConn ~ 4800 5950
-Wire Wire Line
-	4800 3250 5100 3250
 NoConn ~ 4800 5550
+Wire Wire Line
+	3400 4850 3000 4850
+NoConn ~ 3400 5650
+NoConn ~ 4800 3250
 $EndSCHEMATC

Commit message: git :)
Parts:
- removed Y1: Crystal 8Mhz, Crystals:Crystal_SMD_HC49-SD_HandSoldering, symbol Device:Crystal
- added Y1: ECS-80-12-30Q-DS-TR, myLib:Quarz, symbol SamacSys_Parts:ECS-80-12-30Q-DS-TR
Connections:
- net at C1.2, U1.5 (PH0): now also Y1.1 (IN/OUT)
- net at C2.2, U1.6 (PH1): now also Y1.2 (OUT/IN)
Changed lines of the file:
@@
-$EndComp
-$Comp
-L Device:Crystal Y1
-U 1 1 5DC1A7A3
-P 2450 4250
-F 0 "Y1" V 2404 4381 50  0000 L CNN
-F 1 "Crystal 8Mhz" V 2495 4381 50  0000 L CNN
-F 2 "Crystals:Crystal_SMD_HC49-SD_HandSoldering" H 2450 4250 50  0001 C CNN
-F 3 "~" H 2450 4250 50  0001 C CNN
-	1    2450 4250
-	0    1    1    0
 $EndComp
 $Comp
@@
 NoConn ~ 3400 5650
 NoConn ~ 4800 3250
+Wire Wire Line
+	2300 4200 2250 4200
+Wire Wire Line
+	2250 4200 2250 4100
+Wire Wire Line
+	2250 4100 2450 4100
+Wire Wire Line
+	2450 4400 2250 4400
+Wire Wire Line
+	2250 4400 2250 4300
+Wire Wire Line
+	2250 4300 2300 4300
+$Comp
+L SamacSys_Parts:ECS-80-12-30Q-DS-TR Y1
+U 1 1 5DF286AB
+P 2300 4200
+F 0 "Y1" H 3128 4196 50  0000 L CNN
+F 1 "ECS-80-12-30Q-DS-TR" H 3128 4105 50  0000 L CNN
+F 2 "myLib:Quarz" H 3150 4300 50  0001 L CNN
+F 3 "https://componentsearchengine.com/Datasheets/1/ECS-80-12-30Q-DS-TR.pdf" H 3150 4200 50  0001 L CNN
+F 4 "Crystals 8MHz 12pF AEC ESR 100 -40C +125C" H 3150 4100 50  0001 L CNN "Description"
+F 5 "1.1" H 3150 4000 50  0001 L CNN "Height"
+F 6 "520-80-12-30Q-DST" H 3150 3900 50  0001 L CNN "Mouser Part Number"
+F 7 "https://www.mouser.com/Search/Refine.aspx?Keyword=520-80-12-30Q-DST" H 3150 3800 50  0001 L CNN "Mouser Price/Stock"
+F 8 "ECS" H 3150 3700 50  0001 L CNN "Manufacturer_Name"
+F 9 "ECS-80-12-30Q-DS-TR" H 3150 3600 50  0001 L CNN "Manufacturer_Part_Number"
+	1    2300 4200
+	1    0    0    -1
+$EndComp
 $EndSCHEMATC
