File: Schaltplan_embedded/KiCad/ES_proj_LoRaWAN_fsm/Spannungsversorgung.sch (KiCad schematic (older format))
At the start: 38 parts, among them IC1 TLS850B0TBV33ATMA1, IC3 TLS850B0TBV55ATMA1

Commit message: schaltplan neu
Parts:
- L?: value 10u -> 10uH
Changed lines of the file:
@@
 P 2700 800
 F 0 "L?" H 2700 1015 50  0000 C CNN
-F 1 "10u" H 2700 924 50  0000 C CNN
+F 1 "10uH" H 2700 924 50  0000 C CNN
 F 2 "" H 2700 800 50  0001 C CNN
 F 3 "~" H 2700 800 50  0001 C CNN

Commit message: Neuer Schaltplan
Parts:
- C10, C14, C15: footprint (none) -> Capacitors_SMD:C_0603_HandSoldering
- C11, C12, C8: footprint (none) -> Capacitors_SMD:CP_Elec_5x5.3
- C13, C9: footprint (none) -> Capacitors_SMD:C_0805_HandSoldering
- C16, C17, C18, C19, C22, C23, C24: renamed from C?; footprint (none) -> Capacitors_SMD:C_0805_HandSoldering
- C20, C21: renamed from C?; footprint (none) -> Capacitors_SMD:C_0603_HandSoldering
- D2: renamed from D?; footprint STMITE -> (none)
- IC1, IC3: footprint TLS850B0TBV33ATMA1 -> (none)
- IC2: renamed from IC?; footprint QFN50P300X300X100-17N-D -> (none)
- IC4: renamed from IC?; footprint SOP65P640X120-8N -> (none)
- gave numbers to parts that had none: 16
Connections:
- net 3V3 renamed +3V3
- net 5V renamed +5V
Other:
- moved on the sheet: C12, C13, C8, C9

Commit message: Bauteilliste vollständig und Schaltplan entsprechend geändert
Parts:
- removed R16: 0, symbol Device:R
- C10, C14: value 1u -> 1uF
- C11, C15: value 10u -> 10uF
- C12, C8: value 47u -> 47uF
- C13, C9: value 100n -> 100nF
- D2: footprint (none) -> SamacSys_Parts:STMITE
- IC1, IC3: footprint (none) -> SamacSys_Parts:TLS850B0TBV33ATMA1
- IC2: footprint (none) -> SamacSys_Parts:QFN50P300X300X100-17N-D
- IC4: footprint (none) -> SamacSys_Parts:SOP65P640X120-8N
- J2: footprint (none) -> Connect:BARREL_JACK
- J3: footprint (none) -> Pin_Headers:Pin_Header_Straight_1x02_Pitch1.00mm
- L1, R10, R11, R12, R13, R14, R15, R4, R5, R6, R8, R9: footprint (none) -> Resistors_SMD:R_0805_HandSoldering
- R7: footprint (none) -> Resistors_SMD:R_0603_HandSoldering
Other:
- moved on the sheet: C10, C11, C12, C14, C15, C8, C9, L1

Commit message: Schaltplanänderung
Parts:
- removed J2: Barrel_Jack, Connect:BARREL_JACK, symbol Connector:Barrel_Jack
- added J?: CON-SOCJ-2155, CONSOCJ2155, symbol SamacSys_Parts:CON-SOCJ-2155
Changed lines of the file:
@@
-$EndComp
-$Comp
-L Connector:Barrel_Jack J2
-U 1 1 5DD26B6F
-P 1050 1400
-F 0 "J2" H 1105 1725 50  0000 C CNN
-F 1 "Barrel_Jack" H 1105 1634 50  0000 C CNN
-F 2 "Connect:BARREL_JACK" H 1100 1360 50  0001 C CNN
-F 3 "~" H 1100 1360 50  0001 C CNN
-	1    1050 1400
-	1    0    0    -1
 $EndComp
 $Comp
@@
 Wire Wire Line
 	2950 800  2950 1500
+$Comp
+L SamacSys_Parts:CON-SOCJ-2155 J?
+U 1 1 5DE16150
+P 1200 1250
+F 0 "J?" H 1492 869 50  0000 C CNN
+F 1 "CON-SOCJ-2155" H 1492 960 50  0000 C CNN
+F 2 "CONSOCJ2155" H 1850 1100 50  0001 L CNN
+F 3 "http://www.produktinfo.conrad.com/datenblaetter/1500000-1599999/001582350-da-01-en-DC_EINBAUBUCHSE__SCHALTER_GESCHLOSSEN.pdf" H 1850 1000 50  0001 L CNN
+F 4 "DC Power Connectors Power Jack/Connector 2.1mm x 5.5mm" H 1850 900 50  0001 L CNN "Description"
+F 5 "11" H 1850 800 50  0001 L CNN "Height"
+F 6 "992-CON-SOCJ-2155" H 1850 700 50  0001 L CNN "Mouser Part Number"
+F 7 "https://www.mouser.com/Search/Refine.aspx?Keyword=992-CON-SOCJ-2155" H 1850 600 50  0001 L CNN "Mouser Price/Stock"
+F 8 "Gravitech" H 1850 500 50  0001 L CNN "Manufacturer_Name"
+F 9 "CON-SOCJ-2155" H 1850 400 50  0001 L CNN "Manufacturer_Part_Number"
+	1    1200 1250
+	-1   0    0    1
+$EndComp
 $EndSCHEMATC
