File: Schaltplan_embedded/KiCad/ES_proj_LoRaWAN_fsm/Sensorik.sch (KiCad schematic (older format))
At the start: 27 parts, among them IC5 TPS22943DCKR, IC6 BGA824N6E6327XTSA1, IC7 TESEO-LIV3F, J4 CONSMA002-L-G, J5 Conn_01x08_Male, J6 CONSMA002-L-G, U2 RFM92W_93W

Commit message: so
Parts:
- renumbered C27 to C10, C28 to C11, C29 to C12, C30 to C13, C31 to C14, C32 to C15, C33 to C16, C34 to C17, C35 to C18, C36 to C19, C37 to C20, C25 to C8, C26 to C9, D3 to D2, IC5 to IC1, IC6 to IC2, IC7 to IC3, J5 to J3, J6 to J5, L2 to L1, L3 to L2, L4 to L3, R17 to R4, R21 to R5

Commit message: Schaltplan nuevo
Parts:
- removed J3: Conn_01x08_Male, Pin_Headers:Pin_Header_Straight_1x08_Pitch1.00mm, symbol Connector:Conn_01x08_Male
- added J3: 53048-0810, SamacSys_Parts:SHDR8W35P0X125_1X8_1175X550X370P, symbol SamacSys_Parts:53048-0810
- FL1: symbol Schaltplan_embedded-rescue:B4327-RF_Filter_neu -> Schaltplan_embedded-rescue:B4327-RF_Filter_neu-Schaltplan_embedded-rescue
- J4, J5: symbol Schaltplan_embedded-rescue:CONSMA002-L-G-SamacSys_Parts -> Schaltplan_embedded-rescue:CONSMA002-L-G-SamacSys_Parts-Schaltplan_embedded-rescue
- U2: symbol Schaltplan_embedded-rescue:RFM95W-868S2-RF_Module -> Schaltplan_embedded-rescue:RFM95W-868S2-RF_Module-Schaltplan_embedded-rescue
Connections:
- net +5V: now also J3.2
- net GND: now also J3.8
- net UART_4_RX: now also J3.6
- net UART_4_TX: now also J3.7
Changed lines of the file:
@@
 Comment4 ""
 $EndDescr
-NoConn ~ 1350 1050
-NoConn ~ 1350 1250
-NoConn ~ 1350 1350
-NoConn ~ 1350 1450
-Text GLabel 1550 1550 2    50   Input ~ 0
+Text GLabel 1650 1600 2    50   Input ~ 0
 UART_4_RX
-Wire Wire Line
-	1350 1550 1550 1550
-Text GLabel 1550 1650 2    50   Output ~ 0
+Text GLabel 1650 1700 2    50   Output ~ 0
 UART_4_TX
-Wire Wire Line
-	1350 1650 1550 1650
-$Comp
-L Connector:Conn_01x08_Male J3
-U 1 1 5E17DE2D
-P 1150 1350
-F 0 "J3" H 1258 1831 50  0000 C CNN
-F 1 "Conn_01x08_Male" H 1258 1740 50  0000 C CNN
-F 2 "Pin_Headers:Pin_Header_Straight_1x08_Pitch1.00mm" H 1150 1350 50  0001 C CNN
-F 3 "~" H 1150 1350 50  0001 C CNN
-	1    1150 1350
-	1    0    0    -1
-$EndComp
 $Comp
 L power:GND #PWR015
 U 1 1 5E17F498
-P 1500 1850
-F 0 "#PWR015" H 1500 1600 50  0001 C CNN
-F 1 "GND" H 1505 1677 50  0000 C CNN
-F 2 "" H 1500 1850 50  0001 C CNN
-F 3 "" H 1500 1850 50  0001 C CNN
-	1    1500 1850
-	1    0    0    -1
-$EndComp
-Wire Wire Line
-	1350 1750 1500 1750
-Wire Wire Line
-	1500 1750 1500 1850
-Wire Notes Line
-	850  750  850  2100
+P 1600 1850
+F 0 "#PWR015" H 1600 1600 50  0001 C CNN
+F 1 "GND" H 1605 1677 50  0000 C CNN
+F 2 "" H 1600 1850 50  0001 C CNN
+F 3 "" H 1600 1850 50  0001 C CNN
+	1    1600 1850
+	1    0    0    -1
+$EndComp
+Wire Wire Line
+	1600 1800 1600 1850
 Wire Notes Line
 	850  2100 2150 2100
@@
 $EndComp
 $Comp
-L Schaltplan_embedded-rescue:B4327-RF_Filter_neu FL?
+L Schaltplan_embedded-rescue:B4327-RF_Filter_neu-Schaltplan_embedded-rescue FL?
 U 1 1 5DD1B065
 P 7350 4150
@@
 	8300 4150 8650 4150
 $Comp
-L Schaltplan_embedded-rescue:RFM95W-868S2-RF_Module U2
+L Schaltplan_embedded-rescue:RFM95W-868S2-RF_Module-Schaltplan_embedded-rescue U2
 U 1 1 5DE49B3D
 P 2850 6750
@@
 $EndComp
 Wire Wire Line
-	1850 1150 1850 1000
-Wire Wire Line
-	1350 1150 1850 1150
-Wire Wire Line
 	8950 3050 8950 5500
 Wire Wire Line
@@
 	1800 4250 1800 4600
 $Comp
-L Schaltplan_embedded-rescue:CONSMA002-L-G-SamacSys_Parts J5
+L Schaltplan_embedded-rescue:CONSMA002-L-G-SamacSys_Parts-Schaltplan_embedded-rescue J5
 U 1 1 5DDFF1AD
 P 1750 4250
@@
 $EndComp
 $Comp
-L Schaltplan_embedded-rescue:CONSMA002-L-G-SamacSys_Parts J4
+L Schaltplan_embedded-rescue:CONSMA002-L-G-SamacSys_Parts-Schaltplan_embedded-rescue J4
 U 1 1 5DE088FB
 P 1500 6650
@@
 	-1   0    0    1
 $EndComp
+Wire Notes Line
+	850  750  850  2100
+$Comp
+L SamacSys_Parts:53048-0810 J3
+U 1 1 5DEAB6B5
+P 1550 1100
+F 0 "J3" H 1842 1365 50  0000 C CNN
+F 1 "53048-0810" H 1842 1274 50  0000 C CNN
+F 2 "SamacSys_Parts:SHDR8W35P0X125_1X8_1175X550X370P" H 2200 1200 50  0001 L CNN
+F 3 "https://componentsearchengine.com/Datasheets/1/53048-0810.pdf" H 2200 1100 50  0001 L CNN
+F 4 "8 way through board PCB 90deg header Molex PICOBLADE Series, Series Number 53048, 1.25mm Pitch 8 Way 1 Row Right Angle PCB Header, Solder Termination, 1A" H 2200 1000 50  0001 L CNN "Description"
+F 5 "3.7" H 2200 900 50  0001 L CNN "Height"
+F 6 "538-53048-0810" H 2200 800 50  0001 L CNN "Mouser Part Number"
+F 7 "https://www.mouser.com/Search/Refine.aspx?Keyword=538-53048-0810" H 2200 700 50  0001 L CNN "Mouser Price/Stock"
+F 8 "Molex" H 2200 600 50  0001 L CNN "Manufacturer_Name"
+F 9 "53048-0810" H 2200 500 50  0001 L CNN "Manufacturer_Part_Number"
+	1    1550 1100
+	-1   0    0    -1
+$EndComp
+Wire Wire Line
+	1550 1200 1850 1200
+Wire Wire Line
+	1550 1600 1650 1600
+Wire Wire Line
+	1550 1700 1650 1700
+Wire Wire Line
+	1550 1800 1600 1800
+Wire Wire Line
+	1850 1000 1850 1200
+NoConn ~ 1550 1100
+NoConn ~ 1550 1300
+NoConn ~ 1550 1400
+NoConn ~ 1550 1500
 $EndSCHEMATC

Commit message: neuer Schaltplan
Parts:
- removed D2: ESDARF02-1BU2CK, SamacSys_Parts:ESDARF021BU2CK, symbol SamacSys_Parts:ESDARF02-1BU2CK
- added D2: T3V3S5-7, SamacSys_Parts:SODFL1608X65N, symbol SamacSys_Parts:T3V3S5-7
Connections:
- net GND: now also D2.2 (A)
- net at C11.2, J5.5, L1.1: now also D2.1 (K)
Changed lines of the file:
@@
-$EndComp
-$Comp
-L SamacSys_Parts:ESDARF02-1BU2CK D2
-U 1 1 5DD00D5D
-P 2300 4200
-F 0 "D2" V 2654 4328 50  0000 L CNN
-F 1 "ESDARF02-1BU2CK" V 2745 4328 50  0000 L CNN
-F 2 "SamacSys_Parts:ESDARF021BU2CK" H 2950 4300 50  0001 L CNN
-F 3 "https://componentsearchengine.com/Datasheets/1/ESDARF02-1BU2CK.pdf" H 2950 4200 50  0001 L CNN
-F 4 "STMicroelectronics ESDARF02-1BU2CK Bi-Directional ESD Protection Diode, 20W peak, 2-Pin ST-0201" H 2950 4100 50  0001 L CNN "Description"
-F 5 "0.33" H 2950 4000 50  0001 L CNN "Height"
-F 6 "511-ESDARF02-1BU2CK" H 2950 3900 50  0001 L CNN "Mouser Part Number"
-F 7 "https://www.mouser.com/Search/Refine.aspx?Keyword=511-ESDARF02-1BU2CK" H 2950 3800 50  0001 L CNN "Mouser Price/Stock"
-F 8 "STMicroelectronics" H 2950 3700 50  0001 L CNN "Manufacturer_Name"
-F 9 "ESDARF02-1BU2CK" H 2950 3600 50  0001 L CNN "Manufacturer_Part_Number"
-	1    2300 4200
-	0    1    1    0
 $EndComp
 $Comp
@@
 $EndComp
 Wire Wire Line
-	2300 4050 2300 4200
-Wire Wire Line
-	2300 5000 2300 5050
+	2300 4050 2300 4150
+Wire Wire Line
+	2300 4950 2300 5050
 Wire Wire Line
 	2300 5050 2550 5050
@@
 NoConn ~ 1550 1400
 NoConn ~ 1550 1500
+$Comp
+L SamacSys_Parts:T3V3S5-7 D2
+U 1 1 5DF6519C
+P 2300 4150
+F 0 "D2" V 2654 4278 50  0000 L CNN
+F 1 "T3V3S5-7" V 2745 4278 50  0000 L CNN
+F 2 "SamacSys_Parts:SODFL1608X65N" H 2950 4250 50  0001 L CNN
+F 3 "https://componentsearchengine.com/Datasheets/1/T3V3S5-7.pdf" H 2950 4150 50  0001 L CNN
+F 4 "ESD Suppressor TVS 3.3V 2-Pin SOD-523 T/R" H 2950 4050 50  0001 L CNN "Description"
+F 5 "0.65" H 2950 3950 50  0001 L CNN "Height"
+F 6 "621-T3V3S5-7" H 2950 3850 50  0001 L CNN "Mouser Part Number"
+F 7 "https://www.mouser.com/Search/Refine.aspx?Keyword=621-T3V3S5-7" H 2950 3750 50  0001 L CNN "Mouser Price/Stock"
+F 8 "Diodes Inc." H 2950 3650 50  0001 L CNN "Manufacturer_Name"
+F 9 "T3V3S5-7" H 2950 3550 50  0001 L CNN "Manufacturer_Part_Number"
+	1    2300 4150
+	0    1    1    0
+$EndComp
 $EndSCHEMATC

Commit message: Neue platine
Connections:
- net AntOFF: now also IC3.13 (ANT_OFF)
- no-connect marks 11 -> 10
Changed lines of the file:
@@
 Wire Wire Line
 	7950 2000 8200 2000
-NoConn ~ 7950 1800
 $Comp
 L power:GND #PWR014
@@
 	0    1    1    0
 $EndComp
+Text GLabel 8200 1800 2    50   Output ~ 0
+AntOFF
+Wire Wire Line
+	8200 1800 7950 1800
 $EndSCHEMATC

Commit message: git :)
Parts:
- removed C11: 120pF, Capacitors_SMD:C_0805_HandSoldering, symbol Device:C
- removed C18: 1nF, Capacitors_SMD:C_0805, symbol Device:C
- removed C20: 120pF, Capacitors_SMD:C_0805, symbol Device:C
- removed FL1: B4327, SamacSys_Parts:B39162B4353P810, symbol Schaltplan_embedded-rescue:B4327-RF_Filter_neu-Schaltplan_embedded-rescue
- removed IC2: BGA824N6E6327XTSA1, SamacSys_Parts:BGA725L6E6327, symbol SamacSys_Parts:BGA824N6E6327XTSA1
- removed R4: 10k, Resistors_SMD:R_0805_HandSoldering, symbol Device:R
- added C9: 120pF, Capacitor_SMD:C_0805_2012Metric_Pad1.15x1.40mm_HandSolder, symbol Device:C
- C12: value 3.9pF -> 120pF; footprint Capacitors_SMD:C_0805 -> Capacitor_SMD:C_0805_2012Metric_Pad1.15x1.40mm_HandSolder
- C13: renamed from C14; footprint Capacitors_SMD:C_0805 -> Capacitor_SMD:C_0805_2012Metric_Pad1.15x1.40mm_HandSolder
- C14: renamed from C19; footprint Capacitors_SMD:C_0805 -> Capacitor_SMD:C_0805_2012Metric_Pad1.15x1.40mm_HandSolder
- C15: renamed from C17; footprint Capacitors_SMD:C_0805 -> Capacitor_SMD:C_0805_2012Metric_Pad1.15x1.40mm_HandSolder
- C16: renamed from C15; footprint Capacitors_SMD:C_0805 -> Capacitor_SMD:C_0805_2012Metric_Pad1.15x1.40mm_HandSolder
- C17: renamed from C16; footprint Capacitors_SMD:C_0805 -> Capacitor_SMD:C_0805_2012Metric_Pad1.15x1.40mm_HandSolder
- C18: renamed from C13; footprint Capacitors_SMD:C_0805 -> Capacitor_SMD:C_0805_2012Metric_Pad1.15x1.40mm_HandSolder
- L1, L3: footprint Resistors_SMD:R_0805_HandSoldering -> Inductor_SMD:L_0805_2012Metric_Pad1.15x1.40mm_HandSolder
- L2: value 6.8nH -> 100nH; footprint Resistors_SMD:R_0805_HandSoldering -> Inductor_SMD:L_0805_2012Metric_Pad1.15x1.40mm_HandSolder
- renumbered C9 to C10, C10 to C11, IC3 to IC2, R5 to R4
Connections:
- net +3V3: no longer C14.1, IC1.5 (VIN), R4.1
- net GND: now also J4.5, J5.5, L2.2; no longer C12.1, IC2.1 (GND), J4.1, J5.1
- net at D2.1 (K), L1.1: now also C12.2, J5.1; no longer J5.5
- net at L2.1: now also IC2.1 (GND); no longer C12.2
- net at U2.9 (ANT): now also C9.1; no longer J4.5
- net AntOFF: no longer names the net of IC1.4 (ON), IC2.13 (ANT_OFF)
- net RF_IN: no longer names the net of IC2.11 (RF_IN)
- net RF_IN: now also C12.1
- new net: C14.1, IC1.5 (VIN), R4.1
- new net: C9.2, J4.1
Other:
- moved on the sheet: C10, C11, C13, C14, C15, C16, C17, C18, C8, D2, IC1, IC2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
